File: Boards/Suspension_Strain/strain_gauge_circuit.sch (KiCad schematic (older format))
At the start: 0 parts

Commit message: Restore missing contents of file
Parts:
- added C401: C_0.1uF, footprints:C_0805_OEM, symbol Formula:C_0.1uF
- added R101, R102, R103, R104, R105: R_120, footprints:R_0805_OEM, symbol Formula:R_120
- added R106, R407: R_4.99K, footprints:R_0805_OEM, symbol Formula:R_4.99K
- added U101: MCP6001T-I-LT, Package_TO_SOT_SMD:SOT-353_SC-70-5, symbol Formula:MCP6001T-I-LT
Connections:
- new net: R104.1, R106.1, U101.3 (+)
- new net: R105.1, R407.2, U101.4 (-)
- new net: R102.1, R103.2, R105.2
- new net GND: C401.2, R103.1, R106.2, U101.2 (V-)
- new net VCC: C401.1, R101.2, R102.2, U101.5 (V+)
- new net r_strain_+: R101.1, R104.2
- new net strain_gauge_vout: R407.1, U101.1
Other:
- note added: "Strain Gauge Circuit"
